File: hardware/SwanGanzInterface/SGI_PressureChannel2.kicad_sch (KiCad schematic)
At the start: 20 parts, among them J7 Conn_01x04_Pin, U12 INA122D, U13 OPA2350

Commit message: Added footprint and linked to connector symbol
PCB layout also updated with new footprint.
Parts:
- J5: footprint (none) -> Connectors:Pressure_Connector
Changed lines of the file:
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@@
 			)
 		)
-		(property "Footprint" ""
+		(property "Footprint" "Connectors:Pressure_Connector"
 			(at 36.83 62.23 0)
 			(effects
@@
 			)
 		)
-		(property "Footprint" ""
+		(property "Footprint" "Connectors:Pressure_Connector"
 			(at 36.83 97.79 0)
 			(effects
