File: hardware/SwanGanzInterface/SwanGanzInterface.kicad_pcb (KiCad board)
At the start: 2 copper layers, 110 parts, among them J1 2479774-1, J2 Conn_01x08_Pin, J3 Conn_01x03_Pin, J6 Conn_01x04_Pin, J7 Conn_01x04_Pin, Q1 SQ2389CES-T1_GE3, SW1 Power_Switch, SW2 NAV, SW3 ENTER, U1 LM2937ET-3.3_NOPB, U10 INA122D, U11 OPA2350, U12 INA122D, U13 OPA2350, U2 LM4041CILPR, U3 OPA2350, U4 LP-MSPM0G3507, U6 Adafruit ST7735R, U7 FT232R, U8 INA122D, U9 OPA2350

Commit message: Started Layout
Parts:
- removed TP3: +3V3A, SGI_FootprintsLib:Testpoint_1x02_P2.54mm
- removed TP8: DGND, SGI_FootprintsLib:Testpoint_1x02_P2.54mm
- removed TP9: AGND, SGI_FootprintsLib:Testpoint_1x02_P2.54mm
- added U5: AdaFruit_1590, SGI_FootprintsLib:AdaFruit_1590, F.Cu at (68.6, 109.2)
- C10: footprint Capacitor_SMD:C_1206_3216Metric -> Capacitor_SMD:C_0603_1608Metric; moved to B.Cu
- C11: footprint Capacitor_SMD:C_0603_1608Metric -> Capacitor_SMD:C_1206_3216Metric
- C12, C14, C16, C18, C2, C20, C3, C4, C6, C8, C9, Q1, R11, R12, R15, R16, R18, R22, R24, R32, R4, R5: moved to B.Cu
- R29, R36: value 50k -> 10k; moved to B.Cu
- R31, R38: value 10k -> 17k5; moved to B.Cu
- TP2: value +3V3D -> +3V3
- TP6: value DGND -> GND
- TP7: value AGND -> GND
- moved C2 282.0 mm to (35.6, 63.8), turned to -90 degrees
- moved C1 274.1 mm to (45.5, 58.2)
- moved R2 269.1 mm to (36.6, 84.3)
- moved R1 268.8 mm to (36.6, 82.3)
- moved R8 253.4 mm to (42.4, 36.1), turned to 90 degrees
- moved R5 252.3 mm to (139.4, 28.7), turned to -90 degrees
- moved R4 251.2 mm to (136.9, 28.7), turned to 90 degrees
- moved R7 246.2 mm to (42.4, 43.9), turned to 90 degrees
- moved R3 243.2 mm to (137.7, 34.8), turned to 180 degrees
- moved U3 243.1 mm to (143.8, 30.2)
- moved R6 239.2 mm to (42.4, 51.8), turned to 90 degrees
- moved C3 232.4 mm to (147.6, 34.3), turned to -90 degrees
- moved R14 231.1 mm to (61.2, 46.2)
- moved TP4 230.9 mm to (135.9, 37.6), turned to 90 degrees
- moved U7 230.8 mm to (40.1, 104.6), turned to 180 degrees
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Connections:
- D1 pad 1: Net-(D1-K) -> GND
- D2 pad 1: Net-(D1-K) -> GND
- D3 pad 1: Net-(D1-K) -> GND
- TP2 pad 1: +3V3D -> +3V3
- TP2 pad 2: +3V3D -> +3V3
Other:
- board outline added: 127 x 88.9 mm

Commit message: Started Routing
Parts:
- removed TP11, TP12, TP16, TP17, TP21, TP22: TP, SGI_FootprintsLib:Testpoint_1x02_P2.54mm
- added J4: ~, SGI_FootprintsLib:Pressure_Connector, F.Cu at (165.1, 49.5)
- added J5: ~, SGI_FootprintsLib:Pressure_Connector, F.Cu at (165.1, 78.7)
- R17: moved to B.Cu
- R32: moved to F.Cu
- TP10: value TP -> T_InstOut
- TP15: value TP -> P1_InstOut
- TP20: value TP -> P2_InstOut
- moved J2 87.7 mm to (49.7, 68.6), turned to 0 degrees
- moved TP23 66.6 mm to (109.6, 76.7), turned to 90 degrees
- moved TP19 65.1 mm to (110.1, 52.7), turned to 90 degrees
- moved TP18 60.7 mm to (110.1, 47.6), turned to 90 degrees
- moved TP24 50.7 mm to (109.5, 81.8), turned to 90 degrees
- moved TP13 44.8 mm to (133.3, 105.7), turned to 90 degrees
- moved TP14 37.8 mm to (133.3, 100.6), turned to 90 degrees
- moved R17 28.3 mm to (168.8, 98.9), turned to -90 degrees
- moved C11 28.1 mm to (156.8, 100.3)
- moved J3 28.1 mm to (173.0, 100.6)
- moved R15 28.1 mm to (165.2, 103.9)
- moved R16 28.1 mm to (165.2, 101.9)
- moved R18 28.1 mm to (165.2, 105.7)
- moved R19 28.1 mm to (158.3, 103.1)
- moved R20 28.1 mm to (154.5, 103.1)
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Connections:
- J2 pad 6: PB18 -> PA28
- J2 pad 7: PB19 -> PA31
- U4 pad J4_3: unconnected-(U4-PA28-PadJ4_3) -> PA28
- U4 pad J4_4: unconnected-(U4-PA31-PadJ4_4) -> PA31
Routing:
- net PB9: track 0.00 -> 128.8 mm, vias 0 -> 6
- net PB20: track 0.00 -> 67.5 mm, vias 0 -> 3
- net PA31: track 0.00 -> 65.4 mm, vias 0 -> 3
- net PB4: track 0.00 -> 61.1 mm, vias 0 -> 3
- net PA13: track 0.00 -> 54.5 mm
- net PA12: track 0.00 -> 53.2 mm, vias 0 -> 1
- net PA11: track 0.00 -> 52.7 mm, vias 0 -> 1
- net PA10: track 0.00 -> 52.1 mm, vias 0 -> 1
- net PB7: track 0.00 -> 50.9 mm, vias 0 -> 4
- net PB6: track 0.00 -> 40.4 mm, vias 0 -> 4
- net PB15: track 0.00 -> 39.9 mm, vias 0 -> 3
- net PB8: track 0.00 -> 39.6 mm, vias 0 -> 2
- net PB17: track 0.00 -> 37.9 mm, vias 0 -> 3
- net PB16: track 0.00 -> 34.3 mm, vias 0 -> 2
- net PB0: track 0.00 -> 29.1 mm, vias 0 -> 2
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Other:
- board size 127 x 88.9 mm -> 152.4 x 88.9 mm

Commit message: Valvano Changes
Parts:
- D1: value LED -> +3V3
- D2: value LED -> WORKING
- D3: value LED -> ERROR
- moved TP15 11.3 mm to (140.6, 44.6), turned to 90 degrees
- moved R25 2.04 mm to (141.5, 54.7)
- turned R27 to 180 degrees
Routing:
- net ADC_0.2: track 0.00 -> 14.2 mm
- net P1__InstrOut: track 0.00 -> 12.9 mm, vias 0 -> 1
- net ADC_0.3: track 0.00 -> 12.2 mm
- net Net-(U11A-+): track 0.00 -> 6.16 mm
- net Net-(C15-Pad1): track 0.00 -> 4.96 mm
- net Net-(U11B--): track 0.00 -> 4.69 mm
- net P1_SIG-: track 12.6 -> 17.3 mm
- net P1_SIG+: track 22.0 -> 26.4 mm
- net Net-(U11A--): track 0.00 -> 4.29 mm
- net Net-(U10-RG+): track 0.00 -> 4.26 mm
- net Net-(U10-RG-): track 0.00 -> 4.02 mm
- net +VRef: track 22.9 -> 25.5 mm

Commit message: Finished Layout - Requires check and silkscreen
Parts:
- SW2: value NAV -> MODE
- moved TP9 10.5 mm to (143.0, 96.5)
- moved R17 8.20 mm to (176.3, 102.2)
- moved J3 5.02 mm to (172.4, 105.6), turned to 180 degrees
- moved TP15 3.89 mm to (112.4, 84.4), turned to 180 degrees
- moved TP14 2.82 mm to (112.4, 76.7), turned to 180 degrees
- moved R11 2.40 mm to (71.7, 112.3)
- moved JP2 1.55 mm to (75.1, 36.4)
- moved JP1 1.54 mm to (75.1, 32.2)
- moved TP1 0.25 mm to (26.9, 62.0)
- moved TP2 0.25 mm to (26.9, 54.6)
- turned TP10 to 180 degrees
- renumbered J6 to J5, J7 to J6, J5 to J7, TP15 to TP10, TP18 to TP11, TP19 to TP12, TP20 to TP13, TP23 to TP14, TP24 to TP15, TP4 to TP3, TP5 to TP4, TP6 to TP5, TP7 to TP6, TP10 to TP7, TP13 to TP8, TP14 to TP9
Connections:
- C5 pad 1: PB13 -> PB12
- C7 pad 1: PB12 -> PB13
- R10 pad 2: PB13 -> PB12
- R14 pad 2: PB12 -> PB13
- R7 pad 1: PB1 -> PA15
- R8 pad 1: PB2 -> PA16
- U4 pad J1_9: PB2 -> unconnected-(U4-PB2-PadJ1_9)
- U4 pad J3_10: unconnected-(U4-PA15-PadJ3_10) -> PA15
- U4 pad J3_3: PB19 -> unconnected-(U4-PB19-PadJ3_3)
- U4 pad J3_5: PB18 -> unconnected-(U4-PB18-PadJ3_5)
- U4 pad J3_9: unconnected-(U4-PA16-PadJ3_9) -> PA16
- U5 pad 10: PB3 -> PB1
Routing:
- net GND: track 0.00 -> 700.5 mm, vias 0 -> 34
- net +3V3: track 0.00 -> 499.1 mm, vias 0 -> 28
- net +5V: track 0.00 -> 158.2 mm, vias 0 -> 6
- net ADC_0.5: track 14.4 -> 146.2 mm, vias 0 -> 3
- net ADC_0.7: track 12.4 -> 126.4 mm, vias 0 -> 2
- net UART_Tx: track 0.00 -> 101.7 mm, vias 0 -> 5
- net UART_Rx: track 0.00 -> 96.6 mm, vias 0 -> 5
- net PA15: track 0.00 -> 75.0 mm, vias 0 -> 5
- net PB1: track 0.00 -> 74.5 mm, vias 0 -> 4
- net ADC_1.5: track 12.7 -> 82.2 mm, vias 0 -> 4
- net PA16: track 0.00 -> 65.3 mm, vias 0 -> 3
- net ADC_1.3: track 14.7 -> 77.5 mm, vias 0 -> 2
- net ADC_0.2: track 14.2 -> 74.1 mm, vias 0 -> 2
- net PB13: track 0.00 -> 59.8 mm, vias 0 -> 1
- net PA28: track 0.00 -> 50.3 mm, vias 0 -> 3
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Other:
- board text added: "Pressure 1"
- board text added: "Pressure 2"
- board text added: "Thermistor"
