File: hardware/SwanGanzInterface/SwanGanzInterface.kicad_pcb (KiCad board)
At the start: 2 copper layers, 152.4 x 88.9 mm, 104 parts, among them J1 2479774-1, J2 Conn_01x08_Pin, J3 Conn_01x03_Pin, J5 Conn_01x04_Pin, J6 Conn_01x04_Pin, Q1 SQ2389CES-T1_GE3, SW1 Power_Switch, SW2 MODE, SW3 ENTER, U1 LM2937ET-3.3_NOPB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

Commit message: Finished Layout :D
Parts:
- added H1: ~, SGI_FootprintsLib:MountingHole_4_40, F.Cu at (171.4, 31.8)
- added H2: ~, SGI_FootprintsLib:MountingHole_4_40, F.Cu at (119.4, 104.1)
- added H3: ~, SGI_FootprintsLib:MountingHole_4_40, F.Cu at (32.5, 107.1)
- added H4: ~, SGI_FootprintsLib:MountingHole_4_40, F.Cu at (31.1, 31.8)
- added H5: ~, SGI_FootprintsLib:MountingHole_4_40, F.Cu at (142.2, 63.5)
- moved TP4 0.76 mm to (26.9, 71.6)
Routing:
- net GND: track 700.5 -> 698.9 mm
- net +VBUS: track 28.7 -> 29.7 mm
- net +5V: vias 6 -> 5
Other:
- board text added: "S1"

Commit message: Fixed production files
Other:
- board text added: "Ashton Knecht Nathan DeLaRosa Jack Son Jerry Xia Dr. Valvano"
Changed lines of the file:
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@@
 	)
 	(paper "A3")
+	(title_block
+		(comment 1 "Ashton Knecht, Nathan DeLaRosa, Jack Son, Jerry Xia")
+		(comment 2 "Dr. Valvano")
+	)
 	(layers
 		(0 "F.Cu" signal)
@@
 		)
 	)
+	(gr_text "Ashton Knecht\nNathan DeLaRosa\nJack Son\nJerry Xia\nDr. Valvano"
+		(at 111.5568 36.322 0)
+		(layer "F.SilkS")
+		(effects
+			(font
+				(size 1 1)
+				(thickness 0.1)
+			)
+			(justify left bottom)
+		)
+	)
 	(gr_text "Pressure 2"
 		(at 117.602 73.152 0)
@@
 		(layer "B.SilkS")
 		(effects
+			(font
+				(size 1 1)
+				(thickness 0.1)
+			)
+			(justify left bottom mirror)
+		)
+	)
+	(gr_text "Ashton Knecht\nNathan DeLaRosa\nJack Son\nJerry Xia\nDr. Valvano"
+		(at 123.2408 36.322 -0)
+		(layer "B.SilkS")
+		(effects
