File: hardware/SwanGanzInterface/SGI_PressureChannel1.kicad_sch (KiCad schematic)
At the start: 18 parts, among them J5 Conn_01x04_Pin, U10 INA122D, U11 OPA2350

Commit message: Implemented Jack's new pressure footprint and added teardrop - new production file
Parts:
- J4: footprint SGI_FootprintsLib:Pressure_Connector -> SGI_FootprintsLib:Pressure_Connector_1.1
Changed lines of the file:
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@@
 			)
 		)
-		(property "Footprint" "SGI_FootprintsLib:Pressure_Connector"
+		(property "Footprint" "SGI_FootprintsLib:Pressure_Connector_1.1"
 			(at 24.13 62.23 0)
 			(effects
@@
 			)
 		)
-		(property "Footprint" "SGI_FootprintsLib:Pressure_Connector"
+		(property "Footprint" "SGI_FootprintsLib:Pressure_Connector_1.1"
 			(at 24.13 99.06 0)
 			(effects

Commit message: Driver Power
Parts:
- renumbered R25 to R24, R26 to R25, R27 to R26, R28 to R27, R29 to R28, R30 to R29, R31 to R30
Changed lines of the file:
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@@
 		(on_board yes)
 		(dnp no)
-		(property "Reference" "#PWR057"
+		(property "Reference" "#PWR056"
 			(at 146.05 119.38 0)
 			(effects
@@
 			(project "SwanGanzInterface"
 				(path "/4e9a6e30-f660-472b-9696-bea1f34b4545/3d8fa9e7-4833-4941-a955-d778effe3e32"
-					(reference "#PWR057")
+					(reference "#PWR056")
 					(unit 1)
 				)
@@
 		(dnp no)
 		(fields_autoplaced yes)
-		(property "Reference" "#PWR053"
+		(property "Reference" "#PWR052"
 			(at 74.93 46.99 0)
 			(effects
@@
 			(project "SwanGanzInterface"
 				(path "/4e9a6e30-f660-472b-9696-bea1f34b4545/3d8fa9e7-4833-4941-a955-d778effe3e32"
-					(reference "#PWR053")
+					(reference "#PWR052")
 					(unit 1)
 				)
@@
 		(on_board yes)
 		(dnp no)
-		(property "Reference" "R29"
+		(property "Reference" "R28"
 			(at 129.54 71.755 90)
 			(effects
@@
 			(project "SwanGanzInterface"
 				(path "/4e9a6e30-f660-472b-9696-bea1f34b4545/3d8fa9e7-4833-4941-a955-d778effe3e32"
-					(reference "R29")
+					(reference "R28")
 					(unit 1)
 				)
@@
 		(on_board yes)
 		(dnp no)
-		(property "Reference" "#PWR055"
+		(property "Reference" "#PWR054"
 			(at 112.395 81.915 0)
 			(effects
@@
 			(project "SwanGanzInterface"
 				(path "/4e9a6e30-f660-472b-9696-bea1f34b4545/3d8fa9e7-4833-4941-a955-d778effe3e32"
-					(reference "#PWR055")
+					(reference "#PWR054")
 					(unit 1)
 				)
@@
 		(on_board yes)
 		(dnp no)
-		(property "Reference" "R27"
+		(property "Reference" "R26"
 			(at 105.41 60.325 90)
 			(effects
@@
 			(project "SwanGanzInterface"
 				(path "/4e9a6e30-f660-472b-9696-bea1f34b4545/3d8fa9e7-4833-4941-a955-d778effe3e32"
-					(reference "R27")
+					(reference "R26")
 					(unit 1)
 				)
@@
 		(on_board yes)
 		(dnp no)
-		(property "Reference" "#PWR052"
+		(property "Reference" "#PWR051"
 			(at 62.23 88.9 0)
 			(effects
@@
 			(project "SwanGanzInterface"
 				(path "/4e9a6e30-f660-472b-9696-bea1f34b4545/3d8fa9e7-4833-4941-a955-d778effe3e32"
-					(reference "#PWR052")
+					(reference "#PWR051")
 					(unit 1)
 				)
@@
 		(on_board yes)
 		(dnp no)
-		(property "Reference" "#PWR049"
+		(property "Reference" "#PWR048"
 			(at 35.56 199.39 0)
 			(effects
@@
 			(project "SwanGanzInterface"
 				(path "/4e9a6e30-f660-472b-9696-bea1f34b4545/3d8fa9e7-4833-4941-a955-d778effe3e32"
-					(reference "#PWR049")
+					(reference "#PWR048")
 					(unit 1)
 				)
@@
 		(on_board yes)
 		(dnp no)
-		(property "Reference" "#PWR056"
+		(property "Reference" "#PWR055"
 			(at 119.38 93.98 0)
 			(effects
@@
 			(project "SwanGanzInterface"
 				(path "/4e9a6e30-f660-472b-9696-bea1f34b4545/3d8fa9e7-4833-4941-a955-d778effe3e32"
-					(reference "#PWR056")
+					(reference "#PWR055")
 					(unit 1)
 				)
@@
 		(dnp no)
 		(fields_autoplaced yes)
-		(property "Reference" "#PWR059"
+		(property "Reference" "#PWR058"
 			(at 262.89 58.42 0)
 			(effects
@@
 			(project "SwanGanzInterface"
 				(path "/4e9a6e30-f660-472b-9696-bea1f34b4545/3d8fa9e7-4833-4941-a955-d778effe3e32"
-					(reference "#PWR059")
+					(reference "#PWR058")
 					(unit 1)
 				)
@@
 		(on_board yes)
 		(dnp no)
-		(property "Reference" "#PWR051"
+		(property "Reference" "#PWR050"
 			(at 62.23 39.37 0)
 			(effects
@@
 			(project "SwanGanzInterface"
 				(path "/4e9a6e30-f660-472b-9696-bea1f34b4545/3d8fa9e7-4833-4941-a955-d778effe3e32"
-					(reference "#PWR051")
+					(reference "#PWR050")
 					(unit 1)
 				)
@@
 		(on_board yes)
 		(dnp no)
-		(property "Reference" "R30"
+		(property "Reference" "R29"
 			(at 143.764 106.68 90)
 			(effects
@@
 			(project "SwanGanzInterface"
 				(path "/4e9a6e30-f660-472b-9696-bea1f34b4545/3d8fa9e7-4833-4941-a955-d778effe3e32"
-					(reference "R30")
+					(reference "R29")
 					(unit 1)
 				)
@@
 		(on_board yes)
 		(dnp no)
-		(property "Reference" "#PWR050"
+		(property "Reference" "#PWR049"
 			(at 36.83 78.74 0)
 			(effects
@@
 			(project "SwanGanzInterface"
 				(path "/4e9a6e30-f660-472b-9696-bea1f34b4545/3d8fa9e7-4833-4941-a955-d778effe3e32"
-					(reference "#PWR050")
+					(reference "#PWR049")
 					(unit 1)
 				)
@@
 		(on_board yes)
 		(dnp no)
-		(property "Reference" "R25"
+		(property "Reference" "R24"
 			(at 73.66 44.704 90)
 			(effects
@@
 			(project "SwanGanzInterface"
 				(path "/4e9a6e30-f660-472b-9696-bea1f34b4545/3d8fa9e7-4833-4941-a955-d778effe3e32"
-					(reference "R25")
+					(reference "R24")
 					(unit 1)
 				)
@@
 		(on_board yes)
 		(dnp no)
-		(property "Reference" "#PWR054"
+		(property "Reference" "#PWR053"
 			(at 74.93 83.82 0)
 			(effects
@@
 			(project "SwanGanzInterface"
 				(path "/4e9a6e30-f660-472b-9696-bea1f34b4545/3d8fa9e7-4833-4941-a955-d778effe3e32"
-					(reference "#PWR054")
+					(reference "#PWR053")
 					(unit 1)
 				)
@@
 		(on_board yes)
 		(dnp no)
-		(property "Reference" "R31"
+		(property "Reference" "R30"
 			(at 160.02 98.044 90)
 			(effects
@@
 			(project ""
 				(path "/4e9a6e30-f660-472b-9696-bea1f34b4545/3d8fa9e7-4833-4941-a955-d778effe3e32"
-					(reference "R31")
+					(reference "R30")
 					(unit 1)
 				)
@@
 		(on_board yes)
 		(dnp no)
-		(property "Reference" "R28"
+		(property "Reference" "R27"
 			(at 117.475 81.28 90)
 			(effects
@@
 			(project "SwanGanzInterface"
 				(path "/4e9a6e30-f660-472b-9696-bea1f34b4545/3d8fa9e7-4833-4941-a955-d778effe3e32"
-					(reference "R28")
+					(reference "R27")
 					(unit 1)
 				)
@@
 		(on_board yes)
 		(dnp no)
-		(property "Reference" "R26"
+		(property "Reference" "R25"
 			(at 93.98 60.325 90)
 			(effects
@@
 			(project "SwanGanzInterface"
 				(path "/4e9a6e30-f660-472b-9696-bea1f34b4545/3d8fa9e7-4833-4941-a955-d778effe3e32"
-					(reference "R26")
+					(reference "R25")
 					(unit 1)
 				)
@@
 		(on_board yes)
 		(dnp no)
-		(property "Reference" "#PWR058"
+		(property "Reference" "#PWR057"
 			(at 262.89 27.94 0)
 			(effects
@@
 			(project "SwanGanzInterface"
 				(path "/4e9a6e30-f660-472b-9696-bea1f34b4545/3d8fa9e7-4833-4941-a955-d778effe3e32"
-					(reference "#PWR058")
-					(unit 1)
-				)
+					(reference "#PWR057")
+					(unit 1)
+				)
