File: hardware/SwanGanzInterface/SGI_Processor.kicad_sch (KiCad schematic)
At the start: 28 parts, among them J2 Conn_01x08_Pin, SW2 NAV, SW3 ENTER, U4 LP-MSPM0G3507, U5 AdaFruit_1590, U6 Adafruit ST7735R, U7 FT232R

Commit message: Finished Layout - Requires check and silkscreen
Parts:
- SW2: value NAV -> MODE
Connections:
- net PB1: now also U5.10 (WAIT); no longer R7.1
- net PB12: now also C5.1, R10.2; no longer C7.1, R14.2
- net PB13: now also C7.1, R14.2; no longer C5.1, R10.2
- net PB3: no longer U5.10 (WAIT)
- net PA15: now reaches U4.J3_10 (PA15)
- net PA15: now also R7.1
- net PA16: now reaches U4.J3_9 (PA16)
- net PA16: now also R8.1
- net PB18: no longer names the net of U4.J3_5 (PB18)
- net PB19: no longer names the net of U4.J3_3 (PB19)
- net PB2: no longer names the net of U4.J1_9 (PB2)
- net PB2: no longer R8.1
- no-connect marks 28 -> 29
Changed lines of the file:
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@@
 	)
 	(no_connect
-		(at 77.47 63.5)
+		(at 118.11 40.64)
 	)
 	(no_connect
@@
 	)
 	(no_connect
+		(at 118.11 78.74)
+	)
+	(no_connect
 		(at 77.47 45.72)
 	)
@@
 	)
 	(no_connect
+		(at 118.11 43.18)
+	)
+	(no_connect
 		(at 262.89 71.12)
 	)
@@
 	)
 	(no_connect
-		(at 77.47 66.04)
-	)
-	(no_connect
 		(at 262.89 59.69)
 	)
@@
 	(wire
 		(pts
-			(xy 113.03 81.28) (xy 118.11 81.28)
-		)
-		(stroke
-			(width 0)
-			(type default)
-		)
-	)
-	(wire
-		(pts
 			(xy 72.39 54.61) (xy 77.47 54.61)
 		)
@@
 	(wire
 		(pts
-			(xy 113.03 78.74) (xy 118.11 78.74)
-		)
-		(stroke
-			(width 0)
-			(type default)
-		)
-	)
-	(wire
-		(pts
 			(xy 143.51 151.13) (xy 133.35 151.13)
 		)
@@
 	(wire
 		(pts
+			(xy 72.39 66.04) (xy 77.47 66.04)
+		)
+		(stroke
+			(width 0)
+			(type default)
+		)
+	)
+	(wire
+		(pts
 			(xy 38.1 113.03) (xy 43.18 113.03)
 		)
@@
 	(wire
 		(pts
+			(xy 113.03 81.28) (xy 118.11 81.28)
+		)
+		(stroke
+			(width 0)
+			(type default)
+		)
+	)
+	(wire
+		(pts
 			(xy 156.21 168.91) (xy 158.75 168.91)
 		)
@@
 	(wire
 		(pts
+			(xy 118.11 78.74) (xy 113.03 78.74)
+		)
+		(stroke
+			(width 0)
+			(type default)
+		)
+	)
+	(wire
+		(pts
 			(xy 156.21 40.64) (xy 156.21 44.45)
 		)
@@
 	(wire
 		(pts
+			(xy 72.39 63.5) (xy 77.47 63.5)
+		)
+		(stroke
+			(width 0)
+			(type default)
+		)
+	)
+	(wire
+		(pts
 			(xy 179.07 137.16) (xy 179.07 140.97)
 		)
@@
 		)
 	)
-	(global_label "PB1"
+	(global_label "PA15"
 		(shape input)
 		(at 40.64 145.796 90)
@@
 		)
 		(property "Intersheetrefs" "${INTERSHEET_REFS}"
-			(at 40.64 139.0613 90)
+			(at 40.64 138.0332 90)
 			(effects
 				(font
@@
 		)
 	)
+	(global_label "PA15"
+		(shape input)
+		(at 72.39 66.04 180)
+		(fields_autoplaced yes)
+		(effects
+			(font
+				(size 1.27 1.27)
+			)
+			(justify right)
+		)
+		(property "Intersheetrefs" "${INTERSHEET_REFS}"
+			(at 64.6272 66.04 0)
+			(effects
+				(font
+					(size 1.27 1.27)
+				)
+				(justify right)
+				(hide yes)
+			)
+		)
+	)
 	(global_label "PB9"
 		(shape input)
@@
 		)
 	)
-	(global_label "PB19"
-		(shape input)
-		(at 118.11 40.64 0)
-		(fields_autoplaced yes)
-		(effects
-			(font
-				(size 1.27 1.27)
-			)
-			(justify left)
-		)
-		(property "Intersheetrefs" "${INTERSHEET_REFS}"
-			(at 126.0542 40.64 0)
-			(effects
-				(font
-					(size 1.27 1.27)
-				)
-				(justify left)
-				(hide yes)
-			)
-		)
-	)
-	(global_label "PB2"
+	(global_label "PA16"
 		(shape input)
 		(at 52.07 145.796 90)
@@
 		)
 		(property "Intersheetrefs" "${INTERSHEET_REFS}"
-			(at 52.07 139.0613 90)
+			(at 52.07 138.0332 90)
 			(effects
 				(font
@@
 		)
 	)
-	(global_label "PB1"
-		(shape input)
-		(at 118.11 81.28 0)
-		(fields_autoplaced yes)
-		(effects
-			(font
-				(size 1.27 1.27)
-			)
-			(justify left)
-		)
-		(property "Intersheetrefs" "${INTERSHEET_REFS}"
-			(at 124.8447 81.28 0)
-			(effects
-				(font
-					(size 1.27 1.27)
-				)
-				(justify left)
-				(hide yes)
-			)
-		)
-	)
 	(global_label "BACKLITE"
 		(shape input)
@@
 		)
 	)
-	(global_label "PB12"
+	(global_label "PB13"
 		(shape input)
 		(at 207.01 44.45 0)
@@
 		)
 	)
-	(global_label "PB3"
+	(global_label "PB1"
 		(shape input)
 		(at 156.21 172.72 180)
@@
 		)
 	)
+	(global_label "PB1"
+		(shape input)
+		(at 118.11 81.28 0)
+		(fields_autoplaced yes)
+		(effects
+			(font
+				(size 1.27 1.27)
+			)
+			(justify left)
+		)
+		(property "Intersheetrefs" "${INTERSHEET_REFS}"
+			(at 124.8447 81.28 0)
+			(effects
+				(font
+					(size 1.27 1.27)
+				)
+				(justify left)
+				(hide yes)
+			)
+		)
+	)
 	(global_label "PA11"
 		(shape input)
@@
 		)
 	)
-	(global_label "PB18"
-		(shape input)
-		(at 118.11 43.18 0)
-		(fields_autoplaced yes)
-		(effects
-			(font
-				(size 1.27 1.27)
-			)
-			(justify left)
-		)
-		(property "Intersheetrefs" "${INTERSHEET_REFS}"
-			(at 126.0542 43.18 0)
-			(effects
-				(font
-					(size 1.27 1.27)
-				)
-				(justify left)
-				(hide yes)
-			)
-		)
-	)
-	(global_label "PB13"
+	(global_label "PB12"
 		(shape input)
 		(at 171.45 44.45 0)
@@
 		)
 	)
-	(global_label "PB2"
+	(global_label "PA16"
 		(shape input)
-		(at 118.11 78.74 0)
+		(at 72.39 63.5 180)
 		(fields_autoplaced yes)
 		(effects
@@
 				(size 1.27 1.27)
 			)
-			(justify left)
+			(justify right)
 		)
 		(property "Intersheetrefs" "${INTERSHEET_REFS}"
-			(at 124.8447 78.74 0)
+			(at 64.6272 63.5 0)
 			(effects
 				(font
 					(size 1.27 1.27)
 				)
-				(justify left)
+				(justify right)
 				(hide yes)
 			)
@@
 			)
 		)
-		(property "Value" "NAV"
+		(property "Value" "MODE"
 			(at 157.48 54.6099 90)
 			(effects

Commit message: Driver Power
Parts:
- removed R11: 0R, Resistor_SMD:R_0603_1608Metric, symbol Device:R
- renumbered R12 to R11, R13 to R12, R14 to R13
Connections:
- net +3V3: now also C4.1, U5.1 (VIN)
- net +5V: no longer C4.1, U5.1 (VIN)
Changed lines of the file:
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@@
 	)
 	(junction
-		(at 179.07 140.97)
-		(diameter 0)
-		(color 0 0 0 0)
-	)
-	(junction
 		(at 279.4 158.75)
 		(diameter 0)
@@
 	(wire
 		(pts
-			(xy 179.07 137.16) (xy 179.07 140.97)
-		)
-		(stroke
-			(width 0)
-			(type default)
-		)
-	)
-	(wire
-		(pts
 			(xy 204.47 44.45) (xy 204.47 49.53)
 		)
@@
 	(wire
 		(pts
-			(xy 179.07 127) (xy 179.07 129.54)
-		)
-		(stroke
-			(width 0)
-			(type default)
-		)
-	)
-	(wire
-		(pts
 			(xy 72.39 58.42) (xy 77.47 58.42)
 		)
@@
 		(dnp no)
 		(fields_autoplaced yes)
-		(property "Reference" "#PWR029"
+		(property "Reference" "#PWR028"
 			(at 186.69 130.81 0)
 			(effects
@@
 			(project ""
 				(path "/4e9a6e30-f660-472b-9696-bea1f34b4545/b7986f9d-7bcd-462e-9f66-fb6deb5be406"
-					(reference "#PWR029")
+					(reference "#PWR028")
 					(unit 1)
 				)
@@
 			)
 		)
-		(property "Value" "+5V"
-			(at 133.35 128.27 0)
+		(property "Value" "+3V3"
+			(at 135.89 132.0799 0)
 			(effects
 				(font
 					(size 1.27 1.27)
 				)
+				(justify left)
 			)
 		)
@@
 		(dnp no)
 		(fields_autoplaced yes)
-		(property "Reference" "#PWR035"
+		(property "Reference" "#PWR034"
 			(at 279.4 166.37 0)
 			(effects
@@
 			(project ""
 				(path "/4e9a6e30-f660-472b-9696-bea1f34b4545/b7986f9d-7bcd-462e-9f66-fb6deb5be406"
-					(reference "#PWR035")
+					(reference "#PWR034")
 					(unit 1)
 				)
@@
 		(on_board yes)
 		(dnp no)
-		(property "Reference" "R12"
+		(property "Reference" "R11"
 			(at 187.96 130.048 0)
 			(effects
@@
 			(project ""
 				(path "/4e9a6e30-f660-472b-9696-bea1f34b4545/b7986f9d-7bcd-462e-9f66-fb6deb5be406"
-					(reference "R12")
+					(reference "R11")
 					(unit 1)
 				)
@@
 	)
 	(symbol
-		(lib_id "power:+5V")
-		(at 179.07 127 0)
-		(unit 1)
-		(exclude_from_sim no)
-		(in_bom yes)
-		(on_board yes)
-		(dnp no)
-		(fields_autoplaced yes)
-		(property "Reference" "#PWR027"
-			(at 179.07 130.81 0)
-			(effects
-				(font
-					(size 1.27 1.27)
-				)
-				(hide yes)
-			)
-		)
-		(property "Value" "+5V"
-			(at 179.07 121.92 0)
-			(effects
-				(font
-					(size 1.27 1.27)
-				)
-			)
-		)
-		(property "Footprint" ""
-			(at 179.07 127 0)
-			(effects
-				(font
-					(size 1.27 1.27)
-				)
-				(hide yes)
-			)
-		)
-		(property "Datasheet" ""
-			(at 179.07 127 0)
-			(effects
-				(font
-					(size 1.27 1.27)
-				)
-				(hide yes)
-			)
-		)
-		(property "Description" "Power symbol creates a global label with name \"+5V\""
-			(at 179.07 127 0)
-			(effects
-				(font
-					(size 1.27 1.27)
-				)
-				(hide yes)
-			)
-		)
-		(pin "1"
-		)
-		(instances
-			(project ""
-				(path "/4e9a6e30-f660-472b-9696-bea1f34b4545/b7986f9d-7bcd-462e-9f66-fb6deb5be406"
-					(reference "#PWR027")
-					(unit 1)
-				)
-			)
-		)
-	)
-	(symbol
 		(lib_id "SGI_SymbolLib:LED")
 		(at 41.91 165.1 0)
@@
 		(on_board yes)
 		(dnp no)
-		(property "Reference" "R14"
+		(property "Reference" "R13"
 			(at 199.644 42.418 90)
 			(effects
@@
 			(project "SwanGanzInterface"
 				(path "/4e9a6e30-f660-472b-9696-bea1f34b4545/b7986f9d-7bcd-462e-9f66-fb6deb5be406"
-					(reference "R14")
+					(reference "R13")
 					(unit 1)
 				)
@@
 		(dnp no)
 		(fields_autoplaced yes)
-		(property "Reference" "#PWR030"
+		(property "Reference" "#PWR029"
 			(at 191.77 34.29 0)
 			(effects
@@
 			(project "SwanGanzInterface"
 				(path "/4e9a6e30-f660-472b-9696-bea1f34b4545/b7986f9d-7bcd-462e-9f66-fb6deb5be406"
-					(reference "#PWR030")
+					(reference "#PWR029")
 					(unit 1)
 				)
@@
 		(dnp no)
 		(fields_autoplaced yes)
-		(property "Reference" "#PWR034"
+		(property "Reference" "#PWR033"
 			(at 279.4 133.35 0)
 			(effects
@@
 			(project ""
 				(path "/4e9a6e30-f660-472b-9696-bea1f34b4545/b7986f9d-7bcd-462e-9f66-fb6deb5be406"
-					(reference "#PWR034")
+					(reference "#PWR033")
 					(unit 1)
 				)
@@
 		(on_board yes)
 		(dnp no)
-		(property "Reference" "R13"
+		(property "Reference" "R12"
 			(at 193.04 33.02 0)
 			(effects
@@
 			(project "SwanGanzInterface"
 				(path "/4e9a6e30-f660-472b-9696-bea1f34b4545/b7986f9d-7bcd-462e-9f66-fb6deb5be406"
-					(reference "R13")
-					(unit 1)
-				)
-			)
-		)
-	)
-	(symbol
-		(lib_id "Device:R")
-		(at 179.07 133.35 0)
-		(unit 1)
-		(exclude_from_sim no)
-		(in_bom yes)
-		(on_board yes)
-		(dnp no)
-		(property "Reference" "R11"
-			(at 180.086 129.794 0)
-			(effects
-				(font
-					(size 1.27 1.27)
-				)
-				(justify left)
-			)
-		)
-		(property "Value" "0R"
-			(at 179.07 134.62 90)
-			(effects
-				(font
-					(size 1.27 1.27)
-				)
-				(justify left)
-			)
-		)
-		(property "Footprint" "Resistor_SMD:R_0603_1608Metric"
-			(at 177.292 133.35 90)
-			(effects
-				(font
-					(size 1.27 1.27)
-				)
-				(hide yes)
-			)
-		)
-		(property "Datasheet" "~"
-			(at 179.07 133.35 0)
-			(effects
-				(font
-					(size 1.27 1.27)
-				)
-				(hide yes)
-			)
-		)
-		(property "Description" "Resistor"
-			(at 179.07 133.35 0)
-			(effects
-				(font
-					(size 1.27 1.27)
-				)
-				(hide yes)
-			)
-		)
-		(pin "1"
-		)
-		(pin "2"
-		)
-		(instances
-			(project "SwanGanzInterface"
-				(path "/4e9a6e30-f660-472b-9696-bea1f34b4545/b7986f9d-7bcd-462e-9f66-fb6deb5be406"
-					(reference "R11")
+					(reference "R12")
 					(unit 1)
 				)
@@
 		(dnp no)
 		(fields_autoplaced yes)
-		(property "Reference" "#PWR031"
+		(property "Reference" "#PWR030"
 			(at 198.12 69.85 0)
 			(effects
@@
 			(project "SwanGanzInterface"
 				(path "/4e9a6e30-f660-472b-9696-bea1f34b4545/b7986f9d-7bcd-462e-9f66-fb6deb5be406"
-					(reference "#PWR031")
+					(reference "#PWR030")
 					(unit 1)
 				)
@@
 		(dnp no)
 		(fields_autoplaced yes)
-		(property "Reference" "#PWR028"
+		(property "Reference" "#PWR027"
 			(at 179.07 160.02 0)
 			(effects
@@
 			(project ""
 				(path "/4e9a6e30-f660-472b-9696-bea1f34b4545/b7986f9d-7bcd-462e-9f66-fb6deb5be406"
-					(reference "#PWR028")
+					(reference "#PWR027")
 					(unit 1)
 				)
@@
 		(dnp no)
 		(fields_autoplaced yes)
-		(property "Reference" "#PWR032"
+		(property "Reference" "#PWR031"
 			(at 223.52 31.75 0)
 			(effects
@@
 			(project "SwanGanzInterface"
 				(path "/4e9a6e30-f660-472b-9696-bea1f34b4545/b7986f9d-7bcd-462e-9f66-fb6deb5be406"
-					(reference "#PWR032")
+					(reference "#PWR031")
 					(unit 1)
 				)
@@
 		(on_board yes)
 		(dnp no)
-		(property "Reference" "#PWR033"
+		(property "Reference" "#PWR032"
 			(at 236.22 55.88 0)
 			(effects
@@
 			(project "SwanGanzInterface"
 				(path "/4e9a6e30-f660-472b-9696-bea1f34b4545/b7986f9d-7bcd-462e-9f66-fb6deb5be406"
-					(reference "#PWR033")
+					(reference "#PWR032")
 					(unit 1)
 				)
