File: hardware/SwanGanzInterface_V1.1/SGI_Thermistor.kicad_sch (KiCad schematic)
At the start: 20 parts, among them J3 Conn_01x03_Pin, U8 INA122D, U9 OPA2350

Commit message: Pin Allocation, updated schematic with new pins, reassigned
Connections:
- net ADC_0.5 renamed ADC_1.1
- net ADC_0.7 renamed ADC_1.2
Changed lines of the file:
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@@
 		)
 	)
-	(global_label "ADC_0.7"
+	(global_label "ADC_1.2"
 		(shape input)
 		(at 203.2 74.93 0)
@@
 		)
 	)
-	(global_label "ADC_0.5"
+	(global_label "ADC_1.1"
 		(shape input)
 		(at 204.47 53.34 0)

Commit message: Hooked up MSP
Connections:
- net ADC_1.1 renamed THERM_LG_ADC_1.1
- net ADC_1.2 renamed THERM__HG_ADC_1.2
Changed lines of the file:
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@@
 		)
 	)
-	(global_label "ADC_1.2"
+	(global_label "THERM__HG_ADC_1.2"
 		(shape input)
 		(at 203.2 74.93 0)
@@
 		)
 		(property "Intersheetrefs" "${INTERSHEET_REFS}"
-			(at 213.8052 74.93 0)
+			(at 225.477 74.93 0)
 			(effects
 				(font
@@
 		)
 	)
-	(global_label "ADC_1.1"
+	(global_label "THERM_LG_ADC_1.1"
 		(shape input)
 		(at 204.47 53.34 0)
@@
 		)
 		(property "Intersheetrefs" "${INTERSHEET_REFS}"
-			(at 215.0752 53.34 0)
+			(at 225.477 53.34 0)
 			(effects
 				(font

Commit message: Started converting things to use touch screen chip
Connections:
- net THERM_LG_ADC_1.1 renamed THERM_LG_A0.0
- net THERM__HG_ADC_1.2 renamed THERM__HG_A0.1
Changed lines of the file:
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@@
 		)
 	)
-	(global_label "THERM__HG_ADC_1.2"
+	(global_label "THERM__HG_A0.1"
 		(shape input)
 		(at 203.2 74.93 0)
@@
 		)
 		(property "Intersheetrefs" "${INTERSHEET_REFS}"
-			(at 225.477 74.93 0)
+			(at 221.9694 74.93 0)
 			(effects
 				(font
@@
 		)
 	)
-	(global_label "THERM_LG_ADC_1.1"
+	(global_label "THERM_LG_A0.0"
 		(shape input)
 		(at 204.47 53.34 0)
@@
 		)
 		(property "Intersheetrefs" "${INTERSHEET_REFS}"
-			(at 225.477 53.34 0)
+			(at 221.9694 53.34 0)
 			(effects
 				(font
