File: hardware/SwanGanzInterface_V1.1/SGI_PressureChannel1.kicad_sch (KiCad schematic)
At the start: 18 parts, among them J5 Conn_01x04_Pin, U7 INA122D, U8 OPA2350

Commit message: Layout Part 1
Pressure, Audio, Thermistor
Parts:
- removed U7: INA122D, Package_SO:SOIC-8_5.3x5.3mm_P1.27mm, symbol SGI_SymbolLib:INA122D
- added U7: INA122P, Package_DIP:DIP-8_W7.62mm_LongPads, symbol SGI_SymbolLib:INA122P
Connections:
- net +3V3: now also U7.7 (+VS)
- net GND: now also U7.4 (-VS), U7.5 (REF)
- net P1_SIG+: now also U7.3 (+IN)
- net P1_SIG-: now also U7.2 (-IN)
- net P1__InstrOut: now also U7.6 (OUT)
- net at R22.1: now also U7.1 (RG+)
- net at R22.2: now also U7.8 (RG-)
Changed lines of the file:
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@@
+	)
+	(symbol
+		(lib_id "SGI_SymbolLib:INA122P")
+		(at 69.85 62.23 0)
+		(unit 1)
+		(exclude_from_sim no)
+		(in_bom yes)
+		(on_board yes)
+		(dnp no)
+		(property "Reference" "U7"
+			(at 64.3733 80.01 0)
+			(effects
+				(font
+					(size 1.27 1.27)
+				)
+				(justify left)
+			)
+		)
+		(property "Value" "INA122P"
+			(at 60.452 62.23 0)
+			(effects
+				(font
+					(size 1.27 1.27)
+				)
+				(justify left)
+			)
+		)
+		(property "Footprint" "Package_DIP:DIP-8_W7.62mm_LongPads"
+			(at 100.076 68.072 0)
+			(effects
+				(font
+					(size 1.27 1.27)
+				)
+				(hide yes)
+			)
+		)
+		(property "Datasheet" "kicad-embed://ina122.pdf"
+			(at 92.964 66.04 0)
+			(effects
+				(font
+					(size 1.27 1.27)
+				)
+				(hide yes)
+			)
+		)
+		(property "Description" "Instrumentation Amp"
+			(at 89.662 70.104 0)
+			(effects
+				(font
+					(size 1.27 1.27)
+				)
+				(hide yes)
+			)
+		)
+		(pin "8"
+		)
+		(pin "2"
+		)
+		(pin "6"
+		)
+		(pin "5"
+		)
+		(pin "4"
+		)
+		(pin "7"
+		)
+		(pin "3"
+		)
+		(pin "1"
+		)
+		(instances
+			(project "SwanGanzInterface_V1.1"
+				(path "/4e9a6e30-f660-472b-9696-bea1f34b4545/3d8fa9e7-4833-4941-a955-d778effe3e32"
+					(reference "U7")
+					(unit 1)
+				)
+			)
+		)
 	)
 	(symbol
@@
 					(unit 1)
 				)
-			)
-		)
-	)
-	(symbol
-		(lib_id "SGI_SymbolLib:INA122D")
-		(at 69.85 62.23 0)
-		(unit 1)
-		(exclude_from_sim no)
-		(in_bom yes)
-		(on_board yes)
-		(dnp no)
-		(property "Reference" "U7"
-			(at 69.596 62.23 0)
-			(effects
-				(font
-					(size 1.27 1.27)
-				)
-				(justify left)
-			)
-		)
-		(property "Value" "INA122D"
-			(at 69.85 64.008 0)
-			(effects
-				(font
-					(size 1.27 1.27)
-				)
-				(justify left)
-			)
-		)
-		(property "Footprint" "Package_SO:SOIC-8_5.3x5.3mm_P1.27mm"
-			(at 100.076 68.072 0)
-			(effects
-				(font
-					(size 1.27 1.27)
-				)
-				(hide yes)
-			)
-		)
-		(property "Datasheet" "kicad-embed://ina122.pdf"
-			(at 92.964 66.04 0)
-			(effects
-				(font
-					(size 1.27 1.27)
-				)
-				(hide yes)
-			)
-		)
-		(property "Description" "Instrumentation Amp"
-			(at 89.662 70.104 0)
-			(effects
-				(font
-					(size 1.27 1.27)
-				)
-				(hide yes)
-			)
-		)
-		(pin "1"
-		)
-		(pin "8"
-		)
-		(pin "2"
-		)
-		(pin "3"
-		)
-		(pin "7"
-		)
-		(pin "4"
-		)
-		(pin "5"
-		)
-		(pin "6"
-		)
-		(instances
-			(project "SwanGanzInterface"
-				(path "/4e9a6e30-f660-472b-9696-bea1f34b4545/3d8fa9e7-4833-4941-a955-d778effe3e32"
-					(reference "U7")
-					(unit 1)
-				)
