File: hardware/SwanGanzInterface_V1.1/SwanGanzInterface_V1.1.kicad_pcb (KiCad board)
At the start: 4 copper layers, 177.8 x 101.6 mm, 81 parts, among them J12 SPKM.28.8.A, J14 Conn_01x03_Pin, J2 Conn_01x09_Pin, J3 Conn_01x03_Pin, J5 Conn_01x04_Pin, J6 Conn_01x04_Pin, J9 1051640001, U10 OPA2350, U12 MCP34119P, U4 XM0G3507QPMRQ1, U5 INA122P, U6 OPA2350, U7 INA122P, U8 OPA2350, U9 INA122P, Y1 ABM8AIG-40.000MHZ-12-2Z-T3

Commit message: Layout work on screen and expanded board size
Parts:
- added C1: 0.1u, Capacitor_SMD:C_0603_1608Metric, F.Cu at (76.2, 44.2)
- added C11: 0.1u, Capacitor_SMD:C_0603_1608Metric, F.Cu at (270.5, 40.1)
- added C12: 0.1u, Capacitor_SMD:C_0603_1608Metric, F.Cu at (270.5, 42.6)
- added C13: 0.1u, Capacitor_SMD:C_0603_1608Metric, F.Cu at (270.5, 45.1)
- added C2: 10u, Capacitor_SMD:C_1206_3216Metric, B.Cu at (78.7, 44.2)
- added C27: 3.3n, Capacitor_SMD:C_0603_1608Metric, B.Cu at (64.3, 32.8)
- added C28: 0.1u, Capacitor_SMD:C_0603_1608Metric, F.Cu at (284.5, 76.1)
- added C29: 0.1u, Capacitor_SMD:C_0603_1608Metric, F.Cu at (68.1, 54.9)
- added C3: 0.1u, Capacitor_SMD:C_0603_1608Metric, F.Cu at (169.9, 92.2)
- added C30: 4.7u, Capacitor_SMD:C_0805_2012Metric, F.Cu at (68.3, 56.6)
- added C31: 0.1u, Capacitor_SMD:C_0603_1608Metric, F.Cu at (284.5, 81.1)
- added C35: 0.1u, Capacitor_SMD:C_0603_1608Metric, B.Cu at (62.0, 127.8)
- added C37: 1u, Capacitor_SMD:C_0603_1608Metric, F.Cu at (105.4, 127.0)
- added C38: 0.1u, Capacitor_SMD:C_0603_1608Metric, F.Cu at (270.5, 47.6)
- added C39: 0.1u, Capacitor_SMD:C_0603_1608Metric, F.Cu at (270.5, 50.1)
- added C4: 0.1u, Capacitor_SMD:C_0603_1608Metric, F.Cu at (148.3, 95.8)
- added C9: 0.01u, Capacitor_SMD:C_0603_1608Metric, F.Cu at (270.5, 37.6)
- added D1: +3V3, SGI_FootprintsLib:LED_D5.0mm, F.Cu at (34.3, 127.0)
- added D2: WORKING, SGI_FootprintsLib:LED_D5.0mm, F.Cu at (34.3, 111.8)
- added D3: ERROR, SGI_FootprintsLib:LED_D5.0mm, F.Cu at (34.3, 119.4)
- added D4: APHD1608LCGCK, Diode_SMD:D_0603_1608Metric, F.Cu at (74.7, 63.0)
- added D5: APHD1608LSYCK, Diode_SMD:D_0603_1608Metric, F.Cu at (77.3, 63.0)
- added J1: Conn_01x02_Pin, Connector_PinHeader_2.54mm:PinHeader_1x02_P2.54mm_Vertical, F.Cu at (41.5, 35.6)
- added J10: Conn_01x04_Pin, Connector_PinHeader_2.54mm:PinHeader_1x04_P2.54mm_Vertical, F.Cu at (81.8, 34.8)
- added J11: Conn_01x07_Pin, Connector_PinHeader_2.54mm:PinHeader_1x07_P2.54mm_Vertical, F.Cu at (120.1, 136.9)
- added J13: Conn_01x09_Pin, Connector_PinHeader_2.54mm:PinHeader_1x09_P2.54mm_Vertical, F.Cu at (66.0, 136.9)
- added J8: Conn_01x04_Pin, Connector_PinHeader_2.54mm:PinHeader_1x04_P2.54mm_Vertical, F.Cu at (71.2, 34.8)
- added JP1: MicroUSB_VBUS, SGI_FootprintsLib:PinHeader_1x02_P2.54mm_Vertical, F.Cu at (48.3, 41.3)
- added Q1: SQ2389CES-T1_GE3, Package_TO_SOT_SMD:SOT-23, B.Cu at (47.1, 46.7)
- added R1: 47k, Resistor_SMD:R_0603_1608Metric, F.Cu at (162.6, 86.4)
- added R10: 100R, Resistor_SMD:R_0603_1608Metric, F.Cu at (274.5, 50.1)
- added R11: 100R, Resistor_SMD:R_0603_1608Metric, F.Cu at (278.5, 37.6)
- added R2: 10k, Resistor_SMD:R_0603_1608Metric, B.Cu at (162.3, 89.1)
- added R3: 1k, Resistor_SMD:R_0603_1608Metric, B.Cu at (156.2, 88.1)
- added R36: 1M, Resistor_SMD:R_0603_1608Metric, B.Cu at (62.5, 32.8)
- added R37: 2k, Resistor_SMD:R_0603_1608Metric, B.Cu at (39.6, 126.0)
- added R38: 0, Resistor_SMD:R_0603_1608Metric, F.Cu at (287.3, 64.5)
- added R39: 2k, Resistor_SMD:R_0603_1608Metric, B.Cu at (39.6, 111.0)
- added R40: 2k, Resistor_SMD:R_0603_1608Metric, B.Cu at (39.6, 118.4)
- added R41: 750R, Resistor_SMD:R_0603_1608Metric, F.Cu at (83.8, 55.9)
- added R42: 750R, Resistor_SMD:R_0603_1608Metric, F.Cu at (83.8, 58.4)
- added R43: 10k, Resistor_SMD:R_0603_1608Metric, F.Cu at (92.8, 15.6)
- added R44: 19.412k, Resistor_SMD:R_0603_1608Metric, F.Cu at (92.7, 18.5)
- added R45: 100k, Resistor_SMD:R_0603_1608Metric, F.Cu at (112.5, 124.7)
- added R49: 100k, Resistor_SMD:R_0603_1608Metric, F.Cu at (278.5, 40.1)
- added R5: 47k, Resistor_SMD:R_0603_1608Metric, F.Cu at (274.5, 37.6)
- added R50: 100R, Resistor_SMD:R_0603_1608Metric, F.Cu at (278.5, 42.6)
- added R51: 100k, Resistor_SMD:R_0603_1608Metric, F.Cu at (278.5, 45.1)
- added R52: 100R, Resistor_SMD:R_0603_1608Metric, F.Cu at (278.5, 47.6)
- added R6: 100k, Resistor_SMD:R_0603_1608Metric, F.Cu at (274.5, 40.1)
- added R7: 100R, Resistor_SMD:R_0603_1608Metric, F.Cu at (274.5, 42.6)
- added R8: 100k, Resistor_SMD:R_0603_1608Metric, F.Cu at (274.5, 45.1)
- added R9: 100k, Resistor_SMD:R_0603_1608Metric, F.Cu at (274.5, 47.6)
- added SW1: Power_Switch, SGI_FootprintsLib:SW-T3-1A-A-A3-S1, F.Cu at (41.4, 44.2)
- added TP1: +VRef, SGI_FootprintsLib:Testpoint_1x02_P2.54mm, F.Cu at (284.8, 38.7)
- added TP2: +5V, SGI_FootprintsLib:Testpoint_1x02_P2.54mm, F.Cu at (289.5, 38.7)
- added TP3: +3V3, SGI_FootprintsLib:Testpoint_1x02_P2.54mm, F.Cu at (294.1, 38.7)
- added TP4: +VBUS, SGI_FootprintsLib:Testpoint_1x02_P2.54mm, F.Cu at (298.8, 38.7)
- added TP5: GND, SGI_FootprintsLib:Testpoint_1x02_P2.54mm, F.Cu at (303.4, 38.7)
- added TP6: GND, SGI_FootprintsLib:Testpoint_1x02_P2.54mm, F.Cu at (308.1, 38.7)
- added U1: LM4041CILPR, SGI_FootprintsLib:ti_LM4041CILPR, B.Cu at (159.5, 87.4)
- added U11: FT232RNL, SGI_FootprintsLib:FT232RL, F.Cu at (75.9, 56.1)
- added U13: AdaFruit_1590, SGI_FootprintsLib:AdaFruit_1590, F.Cu at (61.0, 130.8)
- added U14: TSC2046IPWR, SGI_FootprintsLib:SOP65P640X120-16N, F.Cu at (105.4, 123.2)
- added U15: LM2937ESX-3.3_NOPB, SGI_FootprintsLib:LM2937ESX-3.3_NOPB, B.Cu at (55.1, 60.0)
- added U2: OPA2350, Package_DIP:DIP-8_W7.62mm, F.Cu at (166.6, 82.0)
- added U3: OPA2350, Package_DIP:DIP-8_W7.62mm, F.Cu at (152.1, 92.5)
- moved J9 83.0 mm to (57.5, 30.1), turned to 0 degrees
- moved H4 18.0 mm to (210.8, 134.6)
- moved J14 12.7 mm to (41.0, 80.3)
- moved J2 12.7 mm to (41.0, 55.4)
- moved C16 12.7 mm to (178.3, 112.9)
- moved C22 12.7 mm to (149.2, 48.9)
- moved C24 12.7 mm to (149.4, 54.9)
- moved C25 12.7 mm to (152.2, 54.9)
- moved C26 12.7 mm to (149.7, 73.1)
- moved J3 12.7 mm to (204.1, 113.3)
- moved J5 12.7 mm to (175.4, 30.0)
- moved J6 12.7 mm to (175.8, 60.8)
- moved J7 12.7 mm to (195.6, 85.8)
- moved R12 12.7 mm to (199.2, 109.4)
- moved R13 12.7 mm to (199.2, 113.2)
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Routing:
- net USB_D-: track 0.00 -> 29.0 mm, vias 0 -> 4
- net MICRO_VBUS: track 0.00 -> 14.1 mm, vias 0 -> 2
- net +VBUS: track 0.00 -> 13.2 mm
Other:
- board size 177.8 x 101.6 mm -> 190.5 x 114.3 mm
- board text added: "CS"
- board text added: "GND"
- board text added: "INT"
- board text added: "LCD Debug"
- board text added: "LITE"
- board text added: "PICO"
- board text added: "POCI"
- board text added: "RST"
- board text added: "SCK"
- board text added: "WAIT"

Commit message: Button pin allocation, layout of power and ft, general layout
Parts:
- added SW2: NRST, SGI_FootprintsLib:SW_PUSH_6mm, F.Cu at (31.8, 95.2)
- added SW3: UP, SGI_FootprintsLib:SW_PUSH_6mm, F.Cu at (134.6, 106.7)
- added SW4: ENTER, SGI_FootprintsLib:SW_PUSH_6mm, F.Cu at (134.6, 116.8)
- added SW5: DOWN, SGI_FootprintsLib:SW_PUSH_6mm, F.Cu at (134.6, 127.0)
- added SW6: LEFT, SGI_FootprintsLib:SW_PUSH_6mm, F.Cu at (121.9, 116.8)
- added SW7: RIGHT, SGI_FootprintsLib:SW_PUSH_6mm, F.Cu at (147.3, 116.8)
- C1, C9, R45, U14: moved to B.Cu
- moved TP5 275.8 mm to (27.6, 38.3)
- moved TP2 262.1 mm to (27.6, 47.8), turned to 180 degrees
- moved TP4 254.0 mm to (45.0, 27.9), turned to 90 degrees
- moved R5 252.1 mm to (30.9, 102.4)
- moved C9 248.7 mm to (29.1, 97.7), turned to 90 degrees
- moved C28 204.5 mm to (81.3, 53.5), turned to 90 degrees
- moved R38 197.3 mm to (92.8, 31.1), turned to -90 degrees
- moved C13 171.3 mm to (137.0, 152.5)
- moved R8 171.3 mm to (141.0, 152.5)
- moved C11 171.3 mm to (137.0, 147.4)
- moved C12 171.3 mm to (137.0, 150.0)
- moved C38 171.3 mm to (137.0, 155.0)
- moved C39 171.3 mm to (137.0, 157.5)
- moved R10 171.3 mm to (141.0, 157.5)
- moved R11 171.3 mm to (145.0, 144.9)
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Connections:
- net Net-(Q1-D) renamed /Power/SW_TO_FET
- C38 pad 1: SW_LEFT_PB20 -> SW_LEFT_PB23
- C39 pad 1: SW_DOWN_PB21 -> SW_DOWN_PB24
- R39 pad 1: LED_WRK_PB23 -> LED_WRK_PA18
- R40 pad 1: LED_ER_PB24 -> LED_ER_PB19
- R50 pad 2: SW_LEFT_PB20 -> SW_LEFT_PB23
- R52 pad 2: SW_DOWN_PB21 -> SW_DOWN_PB24
- U11 pad 12: USB_CBUS4 -> unconnected-(U11-CBUS4-Pad12)
- U4 pad 11: unconnected-(U4-PA18_A1_3-Pad11) -> LED_WRK_PA18
- U4 pad 16: unconnected-(U4-PB19_A1_6-Pad16) -> LED_ER_PB19
- U4 pad 22: LED_WRK_PB23 -> SW_LEFT_PB23
- U4 pad 23: LED_ER_PB24 -> SW_DOWN_PB24
Routing:
- net USB_D+: track 0.00 -> 34.6 mm, vias 0 -> 4
- net +5V: track 0.00 -> 32.7 mm, vias 0 -> 1
- net MICRO_VBUS: track 14.1 -> 31.8 mm
- net FT_+3V3: track 0.00 -> 15.3 mm, vias 0 -> 2
- net USB_D-: track 29.0 -> 40.4 mm
- net +VBUS: track 13.2 -> 24.2 mm, vias 0 -> 2
- net USB_CBUS1: track 0.00 -> 5.77 mm
- net /Power/SW_TO_FET: track 0.00 -> 3.65 mm
- net USB_CBUS0: track 0.00 -> 3.33 mm
- net GND: track 219.9 -> 223.1 mm
Other:
- board text added: "Swan Ganz Interface v2.0 Nathan DeLaRosa Ashton Knecht Jack Son Jerry Xia Dr. Jonathan Valvano"
